File: GlasgowDataIO/Hardware/VacuumController/RPi5VacuumIO/RPi5VacuumIO.kicad_pcb (KiCad board)
At the start: 2 copper layers, 195 x 160 mm, 276 parts, among them J1 24VDC_IN, J11 RELAY1, J12 RELAY2, J13 RELAY3, J14 RELAY4, J15 RELAY5, J16 RELAY6, J17 RELAY7, J18 RELAY8, J2 ESTOP, J21 SOL1-2, J22 SOL3-4, J23 SOL5-6, J24 SOL7-8, J3 RPI5_40PIN, J31 DI1-4, J32 DI5-8, J33 DI9-12, J34 DI13-16, J4 RS485, J41 AI1-4, J42 AI5-8, J5 RS232, K1 G5LE-1 24VDC, K10 G5LE-1 24VDC, K2 G5LE-1 24VDC, K3 G5LE-1 24VDC, K4 G5LE-1 24VDC, K5 G5LE-1 24VDC, K6 G5LE-1 24VDC, K7 G5LE-1 24VDC, K8 G5LE-1 24VDC, K9 G5LE-1 24VDC, Q1 AO3400A, Q2 AO3400A, Q3 AO3400A, Q4 AO3400A, Q5 AO3400A, Q6 AO3400A, Q7 AO3400A, Q8 AO3400A, Q9 AO3400A, U1 MCP23017, U10 ADS1115, U11 MAX3485, U12 MAX3232, U13 TLP291-4, U2 ULN2803A, U3 MCP23017, U5 TLP291-4, U6 TLP291-4, U7 TLP291-4, U8 TLP291-4, U9 ADS1115

Commit message: Re-generate Gerbre | PCB documents
Connections:
- net +24V renamed /+24V
- net +24V_AUX renamed /+24V_AUX
- net +24V_ESTOP renamed /+24V_ESTOP
- net +24V_F renamed /+24V_F
- net +24V_RAW renamed /+24V_RAW
- net +24V_SAFE renamed /+24V_SAFE
- net +3V3 renamed /+3V3
- net ADC_ALRT renamed /ADC_ALRT
- net AI1 renamed /AI1
- net AI2 renamed /AI2
- net AI3 renamed /AI3
- net AI4 renamed /AI4
- net AI5 renamed /AI5
- net AI6 renamed /AI6
- net AI7 renamed /AI7
- net AI8 renamed /AI8
- net AI_S1 renamed /AI_S1
- net AI_S2 renamed /AI_S2
- net AI_S3 renamed /AI_S3
- net AI_S4 renamed /AI_S4
- net AI_S5 renamed /AI_S5
- net AI_S6 renamed /AI_S6
- net AI_S7 renamed /AI_S7
- net AI_S8 renamed /AI_S8
- net C1N renamed /C1N
- net C1P renamed /C1P
- net C2N renamed /C2N
- net C2P renamed /C2P
- net DI1 renamed /DI1
- net DI10 renamed /DI10
- net DI11 renamed /DI11
- net DI12 renamed /DI12
- net DI13 renamed /DI13
- net DI14 renamed /DI14
- net DI15 renamed /DI15
- net DI16 renamed /DI16
- net DI2 renamed /DI2
- net DI3 renamed /DI3
- net DI4 renamed /DI4
- net DI5 renamed /DI5
- net DI6 renamed /DI6
- net DI7 renamed /DI7
- net DI8 renamed /DI8
- net DI9 renamed /DI9
- net DI_A1 renamed /DI_A1
- net DI_A10 renamed /DI_A10
- net DI_A11 renamed /DI_A11
- net DI_A12 renamed /DI_A12
- net DI_A13 renamed /DI_A13
- net DI_A14 renamed /DI_A14
- net DI_A15 renamed /DI_A15
- net DI_A16 renamed /DI_A16
- net DI_A2 renamed /DI_A2
- net DI_A3 renamed /DI_A3
- net DI_A4 renamed /DI_A4
- net DI_A5 renamed /DI_A5
- net DI_A6 renamed /DI_A6
- net DI_A7 renamed /DI_A7
- net DI_A8 renamed /DI_A8
- net DI_A9 renamed /DI_A9
- net DI_COM1 renamed /DI_COM1
- net DI_COM2 renamed /DI_COM2
- net DI_COM3 renamed /DI_COM3
- net DI_COM4 renamed /DI_COM4
- net DI_INT renamed /DI_INT
- net DI_L1 renamed /DI_L1
- net DI_L10 renamed /DI_L10
- net DI_L11 renamed /DI_L11
- net DI_L12 renamed /DI_L12
- net DI_L13 renamed /DI_L13
- net DI_L14 renamed /DI_L14
- net DI_L15 renamed /DI_L15
- net DI_L16 renamed /DI_L16
- net DI_L2 renamed /DI_L2
- net DI_L3 renamed /DI_L3
- net DI_L4 renamed /DI_L4
- net DI_L5 renamed /DI_L5
- net DI_L6 renamed /DI_L6
- net DI_L7 renamed /DI_L7
- net DI_L8 renamed /DI_L8
- net DI_L9 renamed /DI_L9
- net DI_N1 renamed /DI_N1
- net DI_N10 renamed /DI_N10
- net DI_N11 renamed /DI_N11
- net DI_N12 renamed /DI_N12
- net DI_N13 renamed /DI_N13
- net DI_N14 renamed /DI_N14
- net DI_N15 renamed /DI_N15
- net DI_N16 renamed /DI_N16
- net DI_N2 renamed /DI_N2
- net DI_N3 renamed /DI_N3
- net DI_N4 renamed /DI_N4
- net DI_N5 renamed /DI_N5
- net DI_N6 renamed /DI_N6
- net DI_N7 renamed /DI_N7
- net DI_N8 renamed /DI_N8
- net DI_N9 renamed /DI_N9
- net ESTOP_OK_N renamed /ESTOP_OK_N
- net ESTOP_RET renamed /ESTOP_RET
- net GND renamed /GND
- net IO_RESET_N renamed /IO_RESET_N
- net K1_COM renamed /K1_COM
- net K1_NC renamed /K1_NC
- net K1_NO renamed /K1_NO
- net K2_COM renamed /K2_COM
- net K2_NC renamed /K2_NC
- net K2_NO renamed /K2_NO
- net K3_COM renamed /K3_COM
- net K3_NC renamed /K3_NC
- net K3_NO renamed /K3_NO
- net K4_COM renamed /K4_COM
- net K4_NC renamed /K4_NC
- net K4_NO renamed /K4_NO
- net K5_COM renamed /K5_COM
- net K5_NC renamed /K5_NC
- net K5_NO renamed /K5_NO
- net K6_COM renamed /K6_COM
- net K6_NC renamed /K6_NC
- net K6_NO renamed /K6_NO
- net K7_COM renamed /K7_COM
- net K7_NC renamed /K7_NC
- net K7_NO renamed /K7_NO
- net K8_COM renamed /K8_COM
- net K8_NC renamed /K8_NC
- net K8_NO renamed /K8_NO
- net LED_24V renamed /LED_24V
- net LED_EST renamed /LED_EST
- net LED_RUN renamed /LED_RUN
- net LED_SAFE renamed /LED_SAFE
- net RLY_IN1 renamed /RLY_IN1
- net RLY_IN2 renamed /RLY_IN2
- net RLY_IN3 renamed /RLY_IN3
- net RLY_IN4 renamed /RLY_IN4
- net RLY_IN5 renamed /RLY_IN5
- net RLY_IN6 renamed /RLY_IN6
- net RLY_IN7 renamed /RLY_IN7
- net RLY_IN8 renamed /RLY_IN8
- net RLY_L1 renamed /RLY_L1
- net RLY_L2 renamed /RLY_L2
- net RLY_L3 renamed /RLY_L3
- net RLY_L4 renamed /RLY_L4
- net RLY_L5 renamed /RLY_L5
- net RLY_L6 renamed /RLY_L6
- net RLY_L7 renamed /RLY_L7
- net RLY_L8 renamed /RLY_L8
- net RLY_LED1 renamed /RLY_LED1
- net RLY_LED2 renamed /RLY_LED2
- net RLY_LED3 renamed /RLY_LED3
- net RLY_LED4 renamed /RLY_LED4
- net RLY_LED5 renamed /RLY_LED5
- net RLY_LED6 renamed /RLY_LED6
- net RLY_LED7 renamed /RLY_LED7
- net RLY_LED8 renamed /RLY_LED8
- net RLY_V1 renamed /RLY_V1
- net RLY_V2 renamed /RLY_V2
- net RLY_V3 renamed /RLY_V3
- net RLY_V4 renamed /RLY_V4
- net RLY_V5 renamed /RLY_V5
- net RLY_V6 renamed /RLY_V6
- net RLY_V7 renamed /RLY_V7
- net RLY_V8 renamed /RLY_V8
- net RS232_RX renamed /RS232_RX
- net RS232_RXD renamed /RS232_RXD
- net RS232_TX renamed /RS232_TX
- net RS232_TXD renamed /RS232_TXD
- net RS485_A renamed /RS485_A
- net RS485_B renamed /RS485_B
- net RS485_DE renamed /RS485_DE
- net RS485_RX renamed /RS485_RX
- net RS485_T renamed /RS485_T
- net RS485_TX renamed /RS485_TX
- net RUN_LED renamed /RUN_LED
- net SAFE_OK_N renamed /SAFE_OK_N
- net SCL renamed /SCL
- net SDA renamed /SDA
- net SOL_D1 renamed /SOL_D1
- net SOL_D2 renamed /SOL_D2
- net SOL_D3 renamed /SOL_D3
- net SOL_D4 renamed /SOL_D4
- net SOL_D5 renamed /SOL_D5
- net SOL_D6 renamed /SOL_D6
- net SOL_D7 renamed /SOL_D7
- net SOL_D8 renamed /SOL_D8
- net SOL_G1 renamed /SOL_G1
- net SOL_G2 renamed /SOL_G2
- net SOL_G3 renamed /SOL_G3
- net SOL_G4 renamed /SOL_G4
- net SOL_G5 renamed /SOL_G5
- net SOL_G6 renamed /SOL_G6
- net SOL_G7 renamed /SOL_G7
- net SOL_G8 renamed /SOL_G8
- net SOL_IN1 renamed /SOL_IN1
- net SOL_IN2 renamed /SOL_IN2
- net SOL_IN3 renamed /SOL_IN3
- net SOL_IN4 renamed /SOL_IN4
- net SOL_IN5 renamed /SOL_IN5
- net SOL_IN6 renamed /SOL_IN6
- net SOL_IN7 renamed /SOL_IN7
- net SOL_IN8 renamed /SOL_IN8
- net SOL_LED1 renamed /SOL_LED1
- net SOL_LED2 renamed /SOL_LED2
- net SOL_LED3 renamed /SOL_LED3
- net SOL_LED4 renamed /SOL_LED4
- net SOL_LED5 renamed /SOL_LED5
- net SOL_LED6 renamed /SOL_LED6
- net SOL_LED7 renamed /SOL_LED7
- net SOL_LED8 renamed /SOL_LED8
- net ST_A1 renamed /ST_A1
- net ST_A2 renamed /ST_A2
- net VSN renamed /VSN
- net VSP renamed /VSP
- net WDT_AC renamed /WDT_AC
- net WDT_DRAIN renamed /WDT_DRAIN
- net WDT_GATE renamed /WDT_GATE
- net WDT_HB renamed /WDT_HB
- net WDT_HB_R renamed /WDT_HB_R
- J3 pad 11: (no net) -> unconnected-(J3-Pin_11-Pad11)
- J3 pad 18: (no net) -> unconnected-(J3-Pin_18-Pad18)
- J3 pad 19: (no net) -> unconnected-(J3-Pin_19-Pad19)
- J3 pad 2: (no net) -> unconnected-(J3-Pin_2-Pad2)
- J3 pad 21: (no net) -> unconnected-(J3-Pin_21-Pad21)
- J3 pad 22: (no net) -> unconnected-(J3-Pin_22-Pad22)
- J3 pad 23: (no net) -> unconnected-(J3-Pin_23-Pad23)
- J3 pad 24: (no net) -> unconnected-(J3-Pin_24-Pad24)
- J3 pad 26: (no net) -> unconnected-(J3-Pin_26-Pad26)
- J3 pad 27: (no net) -> unconnected-(J3-Pin_27-Pad27)
- J3 pad 28: (no net) -> unconnected-(J3-Pin_28-Pad28)
- J3 pad 36: (no net) -> unconnected-(J3-Pin_36-Pad36)
- J3 pad 38: (no net) -> unconnected-(J3-Pin_38-Pad38)
- J3 pad 4: (no net) -> unconnected-(J3-Pin_4-Pad4)
- J3 pad 40: (no net) -> unconnected-(J3-Pin_40-Pad40)
- J3 pad 7: (no net) -> unconnected-(J3-Pin_7-Pad7)
- K10 pad 3: (no net) -> unconnected-(K10-Pad3)
- K9 pad 3: (no net) -> unconnected-(K9-Pad3)
- U1 pad 11: (no net) -> unconnected-(U1-NC-Pad11)
- U1 pad 14: (no net) -> unconnected-(U1-NC-Pad14)
- U1 pad 19: (no net) -> unconnected-(U1-INTB-Pad19)
- U1 pad 20: (no net) -> unconnected-(U1-INTA-Pad20)
- U12 pad 7: (no net) -> unconnected-(U12-T2OUT-Pad7)
- U12 pad 8: (no net) -> unconnected-(U12-R2IN-Pad8)
- U12 pad 9: (no net) -> unconnected-(U12-R2OUT-Pad9)
- U13 pad 10: (no net) -> unconnected-(U13-Pad10)
- U13 pad 12: (no net) -> unconnected-(U13-Pad12)
- U3 pad 11: (no net) -> unconnected-(U3-NC-Pad11)
- U3 pad 14: (no net) -> unconnected-(U3-NC-Pad14)
- U3 pad 19: (no net) -> unconnected-(U3-INTB-Pad19)
