File: GlasgowDataIO/Hardware/VacuumController/RPi5VacuumIO/RPi5VacuumIO.kicad_sch (KiCad schematic)
At the start: 276 parts, among them J1 24VDC_IN, J11 RELAY1, J12 RELAY2, J13 RELAY3, J14 RELAY4, J15 RELAY5, J16 RELAY6, J17 RELAY7, J18 RELAY8, J2 ESTOP, J21 SOL1-2, J22 SOL3-4, J23 SOL5-6, J24 SOL7-8, J3 RPI5_40PIN, J31 DI1-4, J32 DI5-8, J33 DI9-12, J34 DI13-16, J4 RS485, J41 AI1-4, J42 AI5-8, J5 RS232, K1 G5LE-1 24VDC, K10 G5LE-1 24VDC, K2 G5LE-1 24VDC, K3 G5LE-1 24VDC, K4 G5LE-1 24VDC, K5 G5LE-1 24VDC, K6 G5LE-1 24VDC, K7 G5LE-1 24VDC, K8 G5LE-1 24VDC, K9 G5LE-1 24VDC, Q1 AO3400A, Q2 AO3400A, Q3 AO3400A, Q4 AO3400A, Q5 AO3400A, Q6 AO3400A, Q7 AO3400A, Q8 AO3400A, Q9 AO3400A, U1 MCP23017, U10 ADS1115, U11 MAX3485, U12 MAX3232, U13 TLP291-4, U2 ULN2803A, U3 MCP23017, U5 TLP291-4, U6 TLP291-4, U7 TLP291-4, U8 TLP291-4, U9 ADS1115

Commit message: Re-generate Gerbre | PCB documents
Parts:
- JP1, JP2, JP3, JP4, JP5, JP6, JP7, JP8, JP9: now left out of the parts list
Changed lines of the file:
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@@
     (at 523.24 83.82 0)
     (unit 1)
-    (in_bom yes)
+    (in_bom no)
     (on_board yes)
     (dnp no)
@@
     (at 576.58 83.82 0)
     (unit 1)
-    (in_bom yes)
+    (in_bom no)
     (on_board yes)
     (dnp no)
@@
     (at 632.46 83.82 0)
     (unit 1)
-    (in_bom yes)
+    (in_bom no)
     (on_board yes)
     (dnp no)
@@
     (at 685.8 83.82 0)
     (unit 1)
-    (in_bom yes)
+    (in_bom no)
     (on_board yes)
     (dnp no)
@@
     (at 741.68 83.82 0)
     (unit 1)
-    (in_bom yes)
+    (in_bom no)
     (on_board yes)
     (dnp no)
@@
     (at 797.56 83.82 0)
     (unit 1)
-    (in_bom yes)
+    (in_bom no)
     (on_board yes)
     (dnp no)
@@
     (at 853.44 83.82 0)
     (unit 1)
-    (in_bom yes)
+    (in_bom no)
     (on_board yes)
     (dnp no)
@@
     (at 906.78 83.82 0)
     (unit 1)
-    (in_bom yes)
+    (in_bom no)
     (on_board yes)
     (dnp no)
@@
     (at 401.32 444.5 0)
     (unit 1)
-    (in_bom yes)
+    (in_bom no)
     (on_board yes)
     (dnp no)

Commit message: Update shopping list
Parts:
- J31, J32, J33, J34: MPN Phoenix 1844252 (MC 1,5/6-G-3,5); plug 1840395 -> Phoenix 1844252 (MC 1,5/6-G-3,5); plug 1840405
- J41, J42: MPN Phoenix 1844265 (MC 1,5/8-G-3,5); plug 1840411 -> Phoenix 1844278 (MC 1,5/8-G-3,5); plug 1840421
Changed lines of the file:
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@@
       (at 558.8 274.32 0)
       (effects (font (size 1.27 1.27)) (justify left) hide))
-    (property "MPN" "Phoenix 1844252 (MC 1,5/6-G-3,5); plug 1840395"
+    (property "MPN" "Phoenix 1844252 (MC 1,5/6-G-3,5); plug 1840405"
       (id 4)
       (at 558.8 274.32 0)
@@
       (at 713.74 274.32 0)
       (effects (font (size 1.27 1.27)) (justify left) hide))
-    (property "MPN" "Phoenix 1844252 (MC 1,5/6-G-3,5); plug 1840395"
+    (property "MPN" "Phoenix 1844252 (MC 1,5/6-G-3,5); plug 1840405"
       (id 4)
       (at 713.74 274.32 0)
@@
       (at 868.68 274.32 0)
       (effects (font (size 1.27 1.27)) (justify left) hide))
-    (property "MPN" "Phoenix 1844252 (MC 1,5/6-G-3,5); plug 1840395"
+    (property "MPN" "Phoenix 1844252 (MC 1,5/6-G-3,5); plug 1840405"
       (id 4)
       (at 868.68 274.32 0)
@@
       (at 1026.16 274.32 0)
       (effects (font (size 1.27 1.27)) (justify left) hide))
-    (property "MPN" "Phoenix 1844252 (MC 1,5/6-G-3,5); plug 1840395"
+    (property "MPN" "Phoenix 1844252 (MC 1,5/6-G-3,5); plug 1840405"
       (id 4)
       (at 1026.16 274.32 0)
@@
       (at 299.72 464.82 0)
       (effects (font (size 1.27 1.27)) (justify left) hide))
-    (property "MPN" "Phoenix 1844265 (MC 1,5/8-G-3,5); plug 1840411"
+    (property "MPN" "Phoenix 1844278 (MC 1,5/8-G-3,5); plug 1840421"
       (id 4)
       (at 299.72 464.82 0)
@@
       (at 299.72 487.68 0)
       (effects (font (size 1.27 1.27)) (justify left) hide))
-    (property "MPN" "Phoenix 1844265 (MC 1,5/8-G-3,5); plug 1840411"
+    (property "MPN" "Phoenix 1844278 (MC 1,5/8-G-3,5); plug 1840421"
       (id 4)
       (at 299.72 487.68 0)
